Commit message: fix: rotation and final new line

File: dallara_launch/dallara_description/urdf/dallara.xacro (robot description, xacro)
@@ -6,5 +6,5 @@
   <link name="base_link">
     <visual>
-      <origin xyz="0 0 0" rpy="0 0 0"/>
+      <origin xyz="0 0 0" rpy="0 0 ${pi/2.0}"/>
       <geometry>
         <mesh filename="package://dallara_description/mesh/dallara.dae" scale="1 1 1"/>
